File: schematics/keyer.kicad_sch (KiCad schematic)
At the start: 14 parts, among them J1 Straight Key in, J2 Paddles in, J3 TX Keying out, Q1 2N2222, Q2 2N2222

Commit message: Updates
Other:
- added sheet ESP32 Keyer (ESP32-Keyer.kicad_sch)
Changed lines of the file:
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@@
+    )
+  )
+  (sheet (at 200.66 146.05) (size 31.75 12.7) (fields_autoplaced)
+    (stroke (width 0.1524) (type solid))
+    (fill (color 0 0 0 0.0000))
+    (property "Sheetname" "ESP32 Keyer" (at 200.66 145.3384 0)
+      (effects (font (size 1.27 1.27)) (justify left bottom))
+    )
+    (property "Sheetfile" "ESP32-Keyer.kicad_sch" (at 200.66 159.3346 0)
+      (effects (font (size 1.27 1.27)) (justify left top))
+    )
+    (instances
+      (project "keyer"
+        (path "/985a9195-f593-41f4-969b-dba579e1ad1b" (page "3"))
+      )
     )
   )
